Commit message: sensors complete (step F)

File: body.urdf (robot description, URDF)
Before this commit: robot robot, 3 links, 2 joints
Links:
- removed link Back
- removed link Front
- added link BackLeg, mass 1; collision box size=1 1 1; visual box size=1 1 1
- added link FrontLeg, mass 1; collision box size=1 1 1; visual box size=1 1 1
Joints:
- removed joint Torso_Back
- removed joint Torso_Front
- added joint Torso_BackLeg: type revolute, parent Torso, child BackLeg, origin xyz=-0.5 0 1 rpy=0 0 0, axis 0 1 0, limit lower=-3.14159 upper=3.14159 effort=0.0 velocity=0.0
- added joint Torso_FrontLeg: type revolute, parent Torso, child FrontLeg, origin xyz=0.5 0 1 rpy=0 0 0, axis 0 1 0, limit lower=-3.14159 upper=3.14159 effort=0.0 velocity=0.0

Commit message: Step N Complete

File: body.urdf (robot description, URDF)
Before this commit: robot robot, 3 links, 2 joints
Links:
- added link BackFoot, mass 1; collision box size=0.2 0.2 1; visual box size=0.2 0.2 1
- added link FrontFoot, mass 1; collision box size=0.2 0.2 1; visual box size=0.2 0.2 1
- added link LeftFoot, mass 1; collision box size=0.2 0.2 1; visual box size=0.2 0.2 1
- added link LeftLeg, mass 1; collision box size=1 0.2 0.2; visual box size=1 0.2 0.2
- added link RightFoot, mass 1; collision box size=0.2 0.2 1; visual box size=0.2 0.2 1
- added link RightLeg, mass 1; collision box size=1 0.2 0.2; visual box size=1 0.2 0.2
- link BackLeg: geometry collision box size=0.2 1 0.2; visual box size=0.2 1 0.2
- link FrontLeg: geometry collision box size=0.2 1 0.2; visual box size=0.2 1 0.2
Joints:
- added joint BackLeg_BackFoot: type revolute, parent BackLeg, child BackFoot, origin xyz=0 -0.5 -0.5 rpy=0 0 0, axis 1 0 0, limit lower=-3.14159 upper=3.14159 effort=0.0 velocity=0.0
- added joint FrontLeg_FrontFoot: type revolute, parent FrontLeg, child FrontFoot, origin xyz=0 0.5 -0.5 rpy=0 0 0, axis 1 0 0, limit lower=-3.14159 upper=3.14159 effort=0.0 velocity=0.0
- added joint LeftLeg_LeftFoot: type revolute, parent LeftLeg, child LeftFoot, origin xyz=-0.5 0 -0.5 rpy=0 0 0, axis 0 1 0, limit lower=-3.14159 upper=3.14159 effort=0.0 velocity=0.0
- added joint RightLeg_RightFoot: type revolute, parent RightLeg, child RightFoot, origin xyz=0.5 0 -0.5 rpy=0 0 0, axis 0 1 0, limit lower=-3.14159 upper=3.14159 effort=0.0 velocity=0.0
- added joint Torso_LeftLeg: type revolute, parent Torso, child LeftLeg, origin xyz=-0.5 0 1 rpy=0 0 0, axis 0 1 0, limit lower=-3.14159 upper=3.14159 effort=0.0 velocity=0.0
- added joint Torso_RightLeg: type revolute, parent Torso, child RightLeg, origin xyz=0.5 0 1 rpy=0 0 0, axis 0 1 0, limit lower=-3.14159 upper=3.14159 effort=0.0 velocity=0.0
- joint Torso_BackLeg: axis 0 1 0 -> 1 0 0; origin xyz=-0.5 0 1 rpy=0 0 0 -> xyz=0 -0.5 1 rpy=0 0 0
- joint Torso_FrontLeg: axis 0 1 0 -> 1 0 0; origin xyz=0.5 0 1 rpy=0 0 0 -> xyz=0 0.5 1 rpy=0 0 0

Commit message: Octopod created

File: body.urdf (robot description, URDF)
Before this commit: robot robot, 9 links, 8 joints
Links:
- added link BackFoot2, mass 1; collision box size=0.1 0.6 0.1; visual box size=0.1 0.6 0.1
- added link BackLeg2, mass 1; collision box size=0.2 1 0.2; visual box size=0.2 1 0.2
- added link FrontFoot2, mass 1; collision box size=0.1 0.6 0.1; visual box size=0.1 0.6 0.1
- added link FrontLeg2, mass 1; collision box size=0.2 1 0.2; visual box size=0.2 1 0.2
- added link LeftFoot2, mass 1; collision box size=0.6 0.1 0.1; visual box size=0.6 0.1 0.1
- added link LeftLeg2, mass 1; collision box size=1 0.2 0.2; visual box size=1 0.2 0.2
- added link RightFoot2, mass 1; collision box size=0.6 0.1 0.1; visual box size=0.6 0.1 0.1
- added link RightLeg2, mass 1; collision box size=1 0.2 0.2; visual box size=1 0.2 0.2
- link BackFoot: geometry collision box size=0.1 0.6 0.1; visual box size=0.1 0.6 0.1
- link FrontFoot: geometry collision box size=0.1 0.6 0.1; visual box size=0.1 0.6 0.1
- link LeftFoot: geometry collision box size=0.6 0.1 0.1; visual box size=0.6 0.1 0.1
- link RightFoot: geometry collision box size=0.6 0.1 0.1; visual box size=0.6 0.1 0.1
Joints:
- added joint BackLeg2_BackFoot2: type revolute, parent BackLeg2, child BackFoot2, origin xyz=0 -0.7 0 rpy=0 0 0, axis 1 0 0, limit lower=-3.14159 upper=3.14159 effort=0.0 velocity=0.0
- added joint FrontLeg2_FrontFoot2: type revolute, parent FrontLeg2, child FrontFoot2, origin xyz=0 0.7 0 rpy=0 0 0, axis 1 0 0, limit lower=-3.14159 upper=3.14159 effort=0.0 velocity=0.0
- added joint LeftLeg2_LeftFoot2: type revolute, parent LeftLeg2, child LeftFoot2, origin xyz=-0.7 0 0 rpy=0 0 0, axis 0 1 0, limit lower=-3.14159 upper=3.14159 effort=0.0 velocity=0.0
- added joint RightLeg2_RightFoot2: type revolute, parent RightLeg2, child RightFoot2, origin xyz=0.7 0 0 rpy=0 0 0, axis 0 1 0, limit lower=-3.14159 upper=3.14159 effort=0.0 velocity=0.0
- added joint Torso_BackLeg2: type revolute, parent Torso, child BackLeg2, origin xyz=-0.25 -0.5 0.6 rpy=0 0 0, axis 0 0 1, limit lower=-3.14159 upper=3.14159 effort=0.0 velocity=0.0
- added joint Torso_FrontLeg2: type revolute, parent Torso, child FrontLeg2, origin xyz=-0.25 0.5 0.6 rpy=0 0 0, axis 0 0 1, limit lower=-3.14159 upper=3.14159 effort=0.0 velocity=0.0
- added joint Torso_LeftLeg2: type revolute, parent Torso, child LeftLeg2, origin xyz=-0.5 -0.25 0.6 rpy=0 0 0, axis 0 0 1, limit lower=-3.14159 upper=3.14159 effort=0.0 velocity=0.0
- added joint Torso_RightLeg2: type revolute, parent Torso, child RightLeg2, origin xyz=0.5 -0.25 0.6 rpy=0 0 0, axis 0 0 1, limit lower=-3.14159 upper=3.14159 effort=0.0 velocity=0.0
- joint BackLeg_BackFoot: origin xyz=0 -0.5 -0.5 rpy=0 0 0 -> xyz=0 -0.7 0 rpy=0 0 0
- joint FrontLeg_FrontFoot: origin xyz=0 0.5 -0.5 rpy=0 0 0 -> xyz=0 0.7 0 rpy=0 0 0
- joint LeftLeg_LeftFoot: origin xyz=-0.5 0 -0.5 rpy=0 0 0 -> xyz=-0.7 0 0 rpy=0 0 0
- joint RightLeg_RightFoot: origin xyz=0.5 0 -0.5 rpy=0 0 0 -> xyz=0.7 0 0 rpy=0 0 0
- joint Torso_BackLeg: axis 1 0 0 -> 1 1 1; origin xyz=0 -0.5 1 rpy=0 0 0 -> xyz=0.25 -0.5 0.6 rpy=0 0 0
- joint Torso_FrontLeg: axis 1 0 0 -> 1 1 1; origin xyz=0 0.5 1 rpy=0 0 0 -> xyz=0.25 0.5 0.6 rpy=0 0 0
- joint Torso_LeftLeg: axis 0 1 0 -> 1 1 1; origin xyz=-0.5 0 1 rpy=0 0 0 -> xyz=-0.5 0.25 0.6 rpy=0 0 0
- joint Torso_RightLeg: axis 0 1 0 -> 1 1 1; origin xyz=0.5 0 1 rpy=0 0 0 -> xyz=0.5 0.25 0.6 rpy=0 0 0

Commit message: Random Snakes

File: body.urdf (robot description, URDF)
Before this commit: robot robot, 17 links, 16 joints
Links:
- removed link BackFoot
- removed link BackFoot2
- removed link BackLeg
- removed link BackLeg2
- removed link FrontFoot
- removed link FrontFoot2
- removed link FrontLeg
- removed link FrontLeg2
- removed link LeftFoot
- removed link LeftFoot2
- removed link LeftLeg
- removed link LeftLeg2
- removed link RightFoot
- removed link RightFoot2
- removed link RightLeg
- removed link RightLeg2
- removed link Torso
- added link 0, mass 1; collision box size=1.124661639662299 0.8437931983892348 1.503777981015163; visual box size=1.124661639662299 0.8437931983892348 1.503777981015163
- added link 1, mass 1; collision box size=0.20257996900992714 1.4175572986767644 1.7588610063382188; visual box size=0.20257996900992714 1.4175572986767644 1.7588610063382188
- added link 2, mass 1; collision box size=0.5070199468941821 0.562062153297542 1.0548243073460521; visual box size=0.5070199468941821 0.562062153297542 1.0548243073460521
- added link 3, mass 1; collision box size=1.0515838206916013 0.9900783166356182 1.741128196929069; visual box size=1.0515838206916013 0.9900783166356182 1.741128196929069
- added link 4, mass 1; collision box size=0.919680669630764 0.453303070246431 0.9199192077900877; visual box size=0.919680669630764 0.453303070246431 0.9199192077900877
- added link 5, mass 1; collision box size=0.7986431540612757 1.6249110410311163 0.8910293790451747; visual box size=0.7986431540612757 1.6249110410311163 0.8910293790451747
- added link 6, mass 1; collision box size=0.12378224339097212 1.1183044910094482 0.4618571616733092; visual box size=0.12378224339097212 1.1183044910094482 0.4618571616733092
Joints:
- removed joint BackLeg2_BackFoot2
- removed joint BackLeg_BackFoot
- removed joint FrontLeg2_FrontFoot2
- removed joint FrontLeg_FrontFoot
- removed joint LeftLeg2_LeftFoot2
- removed joint LeftLeg_LeftFoot
- removed joint RightLeg2_RightFoot2
- removed joint RightLeg_RightFoot
- removed joint Torso_BackLeg
- removed joint Torso_BackLeg2
- removed joint Torso_FrontLeg
- removed joint Torso_FrontLeg2
- removed joint Torso_LeftLeg
- removed joint Torso_LeftLeg2
- removed joint Torso_RightLeg
- removed joint Torso_RightLeg2
- added joint 0_1: type revolute, parent 0, child 1, origin xyz=0.5623308198311495 0 0.4397152515845547 rpy=0 0 0, axis 0 1 0, limit lower=-3.14159 upper=3.14159 effort=0.0 velocity=0.0
- added joint 1_2: type revolute, parent 1, child 2, origin xyz=0.20257996900992714 0 0 rpy=0 0 0, axis 0 1 0, limit lower=-3.14159 upper=3.14159 effort=0.0 velocity=0.0
- added joint 2_3: type revolute, parent 2, child 3, origin xyz=0.5070199468941821 0 0 rpy=0 0 0, axis 0 1 0, limit lower=-3.14159 upper=3.14159 effort=0.0 velocity=0.0
- added joint 3_4: type revolute, parent 3, child 4, origin xyz=1.0515838206916013 0 0 rpy=0 0 0, axis 0 1 0, limit lower=-3.14159 upper=3.14159 effort=0.0 velocity=0.0
- added joint 4_5: type revolute, parent 4, child 5, origin xyz=0.919680669630764 0 0 rpy=0 0 0, axis 0 1 0, limit lower=-3.14159 upper=3.14159 effort=0.0 velocity=0.0
- added joint 5_6: type revolute, parent 5, child 6, origin xyz=0.7986431540612757 0 0 rpy=0 0 0, axis 0 1 0, limit lower=-3.14159 upper=3.14159 effort=0.0 velocity=0.0

Commit message: pre-full run

File: body.urdf (robot description, URDF)
Before this commit: robot robot, 7 links, 6 joints
Links:
- added link 10, mass 1; collision box size=1.7399523864775928 1.012372087800642 0.6614963440850428; visual box size=1.7399523864775928 1.012372087800642 0.6614963440850428
- added link 11, mass 1; collision box size=0.3190247442497112 0.2345059237348307 1.6468262724570297; visual box size=0.3190247442497112 0.2345059237348307 1.6468262724570297
- added link 7, mass 1; collision box size=0.9125253393245583 0.8656209483356475 0.9329631043924609; visual box size=0.9125253393245583 0.8656209483356475 0.9329631043924609
- added link 8, mass 1; collision box size=0.5664737779212001 0.6190356014499725 0.3051591485566278; visual box size=0.5664737779212001 0.6190356014499725 0.3051591485566278
- added link 9, mass 1; collision box size=1.2857933927067622 1.1016723932266568 1.8534703519652862; visual box size=1.2857933927067622 1.1016723932266568 1.8534703519652862
- link 0: geometry collision box size=0.5 0.5 0.5; visual box size=0.5 0.5 0.5
- link 1: geometry collision box size=0.1826953310719457 1.1119477481319464 1.2031785237401091; visual box size=0.1826953310719457 1.1119477481319464 1.2031785237401091
- link 2: geometry collision box size=0.9125253393245583 0.8656209483356475 0.9329631043924609; visual box size=0.9125253393245583 0.8656209483356475 0.9329631043924609
- link 3: geometry collision box size=0.5664737779212001 0.6190356014499725 0.3051591485566278; visual box size=0.5664737779212001 0.6190356014499725 0.3051591485566278
- link 4: geometry collision box size=1.2857933927067622 1.1016723932266568 1.8534703519652862; visual box size=1.2857933927067622 1.1016723932266568 1.8534703519652862
- link 5: geometry collision box size=1.7399523864775928 1.012372087800642 0.6614963440850428; visual box size=1.7399523864775928 1.012372087800642 0.6614963440850428
- link 6: geometry collision box size=0.3190247442497112 0.2345059237348307 1.6468262724570297; visual box size=0.3190247442497112 0.2345059237348307 1.6468262724570297
Joints:
- added joint 10_11: type revolute, parent 10, child 11, origin xyz=-0.8699761932387964 0.506186043900321 0 rpy=0 0 0, axis 1 1 1, limit lower=-3.14159 upper=3.14159 effort=0.0 velocity=0.0
- added joint 1_7: type revolute, parent 1, child 7, origin xyz=0.09134766553597284 0.5559738740659732 0 rpy=0 0 0, axis 1 1 1, limit lower=-3.14159 upper=3.14159 effort=0.0 velocity=0.0
- added joint 7_8: type revolute, parent 7, child 8, origin xyz=-0.45626266966227913 0 -0.46648155219623044 rpy=0 0 0, axis 1 1 1, limit lower=-3.14159 upper=3.14159 effort=0.0 velocity=0.0
- added joint 8_9: type revolute, parent 8, child 9, origin xyz=-0.28323688896060006 0 -0.1525795742783139 rpy=0 0 0, axis 1 1 1, limit lower=-3.14159 upper=3.14159 effort=0.0 velocity=0.0
- added joint 9_10: type revolute, parent 9, child 10, origin xyz=-1.2857933927067622 0 0 rpy=0 0 0, axis 1 1 1, limit lower=-3.14159 upper=3.14159 effort=0.0 velocity=0.0
- joint 0_1: axis 0 1 0 -> 1 1 1; origin xyz=0.5623308198311495 0 0.4397152515845547 rpy=0 0 0 -> xyz=0.25 0 3 rpy=0 0 0
- joint 1_2: axis 0 1 0 -> 1 1 1; origin xyz=0.20257996900992714 0 0 rpy=0 0 0 -> xyz=0.09134766553597284 -0.5559738740659732 0 rpy=0 0 0
- joint 2_3: axis 0 1 0 -> 1 1 1; origin xyz=0.5070199468941821 0 0 rpy=0 0 0 -> xyz=-0.45626266966227913 0 -0.46648155219623044 rpy=0 0 0
- joint 3_4: axis 0 1 0 -> 1 1 1; origin xyz=1.0515838206916013 0 0 rpy=0 0 0 -> xyz=-0.28323688896060006 0 -0.1525795742783139 rpy=0 0 0
- joint 4_5: axis 0 1 0 -> 1 1 1; origin xyz=0.919680669630764 0 0 rpy=0 0 0 -> xyz=-1.2857933927067622 0 0 rpy=0 0 0
- joint 5_6: axis 0 1 0 -> 1 1 1; origin xyz=0.7986431540612757 0 0 rpy=0 0 0 -> xyz=-0.8699761932387964 -0.506186043900321 0 rpy=0 0 0
