Commit message: Complete run

File: bodies/9seedbody1653.urdf (robot description, URDF)
Before this commit: robot robot, 12 links, 11 joints
Links:
- link 1: geometry collision box size=0.5091303644759453 0.43542514963453344 0.6958858500830727; visual box size=0.5091303644759453 0.43542514963453344 0.6958858500830727
- link 10: geometry collision box size=1.243306903440335 1.1965807564613304 1.472873418506685; visual box size=1.243306903440335 1.1965807564613304 1.472873418506685
- link 11: geometry collision box size=0.9295510284188291 0.14752681946829826 1.2679040811889424; visual box size=0.9295510284188291 0.14752681946829826 1.2679040811889424
- link 2: geometry collision box size=0.43600697865261856 0.017543095453303452 1.2916951896709215; visual box size=0.43600697865261856 0.017543095453303452 1.2916951896709215
- link 3: geometry collision box size=1.7504859118848284 0.32622430788063317 0.8225119642046818; visual box size=1.7504859118848284 0.32622430788063317 0.8225119642046818
- link 4: geometry collision box size=0.8530556865217345 0.023322012264718632 1.0869783737017475; visual box size=0.8530556865217345 0.023322012264718632 1.0869783737017475
- link 5: geometry collision box size=1.243306903440335 1.1965807564613304 1.472873418506685; visual box size=1.243306903440335 1.1965807564613304 1.472873418506685
- link 6: geometry collision box size=0.9295510284188291 0.14752681946829826 1.2679040811889424; visual box size=0.9295510284188291 0.14752681946829826 1.2679040811889424
- link 7: geometry collision box size=0.43600697865261856 0.017543095453303452 1.2916951896709215; visual box size=0.43600697865261856 0.017543095453303452 1.2916951896709215
- link 8: geometry collision box size=1.7504859118848284 0.32622430788063317 0.8225119642046818; visual box size=1.7504859118848284 0.32622430788063317 0.8225119642046818
- link 9: geometry collision box size=0.8530556865217345 0.023322012264718632 1.0869783737017475; visual box size=0.8530556865217345 0.023322012264718632 1.0869783737017475
Joints:
- joint 10_11: origin xyz=-0.8699761932387964 0.506186043900321 0 rpy=0 0 0 -> xyz=-1.243306903440335 0 0 rpy=0 0 0
- joint 1_2: origin xyz=0.09134766553597284 -0.5559738740659732 0 rpy=0 0 0 -> xyz=0.25456518223797264 -0.21771257481726672 0 rpy=0 0 0
- joint 1_7: origin xyz=0.09134766553597284 0.5559738740659732 0 rpy=0 0 0 -> xyz=0.25456518223797264 0.21771257481726672 0 rpy=0 0 0
- joint 2_3: origin xyz=-0.45626266966227913 0 -0.46648155219623044 rpy=0 0 0 -> xyz=0 0 -1.2916951896709215 rpy=0 0 0
- joint 3_4: origin xyz=-0.28323688896060006 0 -0.1525795742783139 rpy=0 0 0 -> xyz=0 0 -0.8225119642046818 rpy=0 0 0
- joint 4_5: origin xyz=-1.2857933927067622 0 0 rpy=0 0 0 -> xyz=-0.42652784326086723 0 -0.5434891868508738 rpy=0 0 0
- joint 5_6: origin xyz=-0.8699761932387964 -0.506186043900321 0 rpy=0 0 0 -> xyz=-1.243306903440335 0 0 rpy=0 0 0
- joint 7_8: origin xyz=-0.45626266966227913 0 -0.46648155219623044 rpy=0 0 0 -> xyz=0 0 -1.2916951896709215 rpy=0 0 0
- joint 8_9: origin xyz=-0.28323688896060006 0 -0.1525795742783139 rpy=0 0 0 -> xyz=0 0 -0.8225119642046818 rpy=0 0 0
- joint 9_10: origin xyz=-1.2857933927067622 0 0 rpy=0 0 0 -> xyz=-0.42652784326086723 0 -0.5434891868508738 rpy=0 0 0
